Commit message: unknown changes from a while ago. need to investigate

File: models/test/KrangBlocksHands_basewheel.urdf (robot description, URDF)
Before this commit: robot Krang, 3 links, 2 joints
Links:
- removed link RWheel
- link Base: geometry visual box size=0.7165 0.71048 0.32860
- link LWheel: geometry visual mesh filename=Base/oldwheel.dae
Joints:
- removed joint JRWheel
